File: Hardware/PCB/PCB.kicad_pcb (KiCad board)
At the start: 2 copper layers, 32.7 x 35.7 mm, 21 parts, among them J1 USB_C_Receptacle_USB2.0_14P, J2 Conn_01x08_Pin, J3 Conn_01x8_Pin, SW1 SW_Push, SW2 SW_Push, U1 ESP32-H2-MINI-1, U3 MCP1700x-330xxTT

Commit message: Made some corrections. PCB layout needs updating!
Parts:
- added R7: 10K, Resistor_SMD:R_0805_2012Metric, F.Cu at (115.3, 45.0)
- added R8: 10K, Resistor_SMD:R_0805_2012Metric, F.Cu at (83.3, 46.0)
Connections:
- J3 pad 4: GPIO9 -> GPIO0
- U1 pad 23: GPIO9 -> BOOT
- U1 pad 9: BOOT -> GPIO0
Routing:
- net GPIO0: track 0.00 -> 23.9 mm, vias 0 -> 2
- net GPIO9: track 13.4 -> 0.00 mm
- net GPIO8: track 13.5 -> 24.9 mm, vias 0 -> 2
- net BOOT: track 33.8 -> 24.4 mm
- net GND: track 108.5 -> 110.0 mm, vias 6 -> 7
