File: Hardware/PCB/PCB.kicad_sch (KiCad schematic)
At the start: 21 parts, among them J1 USB_C_Receptacle_USB2.0_14P, J2 Conn_01x08_Pin, J3 Conn_01x8_Pin, SW1 SW_Push, SW2 SW_Push, U1 ESP32-H2-MINI-1, U3 MCP1700x-330xxTT

Commit message: Made some corrections. PCB layout needs updating!
Parts:
- added R7, R8: 10K, Resistor_SMD:R_0805_2012Metric, symbol Device:R
Connections:
- net +3.3V: now also R8.1
- net BOOT: now also U1.23 (GPIO9); no longer U1.9 (GPIO0/FSPIQ)
- net GND: now also R7.2
- net GPIO8: now also R7.1, R8.2
- net GPIO9 renamed GPIO0
- net GPIO0: now also U1.9 (GPIO0/FSPIQ); no longer U1.23 (GPIO9)
